File: Modulator/modulator.kicad_pcb (KiCad board)
At the start: 2 copper layers, 78 x 94 mm, 44 parts, among them K1 CONN_20, P1 CONN_1, P2 CONN_1, T1 KC509, X1 4,43MHz

Commit message: Modulator update
Parts:
- R14: value 82R -> 2R2
- TR1: value POT -> 470R
Connections:
- net //BURST renamed //BURST
- net //RSI renamed //RSI
- net //RZI renamed //RZI
- net //SSYN renamed //SSYN
- net /H/2 renamed /H/2
- IO2 pad 15: (no net) -> unconnected-(IO2-Pad15)
- K1 pad 3: Net-(K1-Pad3) -> unconnected-(K1-Pad3)
