File: Modulator/modulator.kicad_sch (KiCad schematic)
At the start: 43 parts, among them K1 CONN_20, P1 CONN_1, P2 CONN_1, T1 KC509, X1 4,43MHz

Commit message: Modulator update
Parts:
- R14: value 82R -> 2R2
Changed lines of the file:
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@@
     (in_bom yes) (on_board yes)
     (property "Reference" "R14" (id 0) (at 241.3 103.378 90))
-    (property "Value" "82R" (id 1) (at 241.3 105.41 90))
+    (property "Value" "2R2" (id 1) (at 241.3 105.41 90))
     (property "Footprint" "" (id 2) (at 241.3 105.41 0)
       (effects (font (size 1.27 1.27)) hide)
@@
     )
     (path "/00000000-0000-0000-0000-00004f51338b"
-      (reference "R14") (unit 1) (value "82R") (footprint "")
+      (reference "R14") (unit 1) (value "2R2") (footprint "")
     )
     (path "/00000000-0000-0000-0000-00004f5132c4"
